File: prototypes/tanksensor/tanksensor/1wire.kicad_sch (KiCad schematic)
At the start: 2 parts, among them J4 Conn_01x03

Commit message: Rev of the tanksensor pcb and esphome config
Parts:
- added D8, D9: D_TVS_30V, Diode_SMD:D_SOD-123F, symbol Device:D_TVS
Connections:
- net +5V: now also D8.1 (A1)
- net DQ_OUT: now also D9.1 (A1)
- net GND: now also D8.2 (A2), D9.2 (A2)
Other:
- moved on the sheet: R8
Changed lines of the file:
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@@
 (kicad_sch (version 20211123) (generator eeschema)
   (paper "A4")
-  (junction (at 109.855 81.28) (diameter 0) (color 0 0 0 0)
-  )
-  (junction (at 109.855 68.58) (diameter 0) (color 0 0 0 0)
+  (junction (at 116.205 81.28) (diameter 0) (color 0 0 0 0)
+  )
+  (junction (at 116.205 68.58) (diameter 0) (color 0 0 0 0)
+  )
+  (junction (at 99.695 68.58) (diameter 0) (color 0 0 0 0)
+  )
+  (junction (at 83.82 101.6) (diameter 0) (color 0 0 0 0)
+  )
+  (junction (at 83.82 81.28) (diameter 0) (color 0 0 0 0)
   )
   (wire (pts (xy 226.06 41.91) (xy 219.71 41.91))
@@
     (stroke (width 0) (type default) (color 0 0 0 0))
   )
-  (wire (pts (xy 79.375 81.28) (xy 109.855 81.28))
-    (stroke (width 0) (type default) (color 0 0 0 0))
-  )
-  (wire (pts (xy 109.855 78.74) (xy 109.855 81.28))
-    (stroke (width 0) (type default) (color 0 0 0 0))
-  )
-  (wire (pts (xy 109.855 68.58) (xy 109.855 71.12))
+  (wire (pts (xy 79.375 81.28) (xy 83.82 81.28))
+    (stroke (width 0) (type default) (color 0 0 0 0))
+  )
+  (wire (pts (xy 116.205 78.74) (xy 116.205 81.28))
+    (stroke (width 0) (type default) (color 0 0 0 0))
+  )
+  (wire (pts (xy 83.82 81.28) (xy 116.205 81.28))
+    (stroke (width 0) (type default) (color 0 0 0 0))
+  )
+  (wire (pts (xy 116.205 68.58) (xy 116.205 71.12))
+    (stroke (width 0) (type default) (color 0 0 0 0))
+  )
+  (wire (pts (xy 99.695 98.425) (xy 99.695 101.6))
+    (stroke (width 0) (type default) (color 0 0 0 0))
+  )
+  (wire (pts (xy 99.695 68.58) (xy 116.205 68.58))
     (stroke (width 0) (type default) (color 0 0 0 0))
   )
@@
     (stroke (width 0) (type default) (color 0 0 0 0))
   )
-  (wire (pts (xy 109.855 81.28) (xy 154.94 81.28))
-    (stroke (width 0) (type default) (color 0 0 0 0))
-  )
-  (wire (pts (xy 109.855 68.58) (xy 160.02 68.58))
+  (wire (pts (xy 99.695 68.58) (xy 99.695 90.805))
     (stroke (width 0) (type default) (color 0 0 0 0))
   )
@@
     (stroke (width 0) (type default) (color 0 0 0 0))
   )
+  (wire (pts (xy 83.82 81.28) (xy 83.82 90.805))
+    (stroke (width 0) (type default) (color 0 0 0 0))
+  )
   (wire (pts (xy 46.99 71.12) (xy 79.375 71.12))
     (stroke (width 0) (type default) (color 0 0 0 0))
@@
     (stroke (width 0) (type default) (color 0 0 0 0))
   )
+  (wire (pts (xy 99.695 101.6) (xy 83.82 101.6))
+    (stroke (width 0) (type default) (color 0 0 0 0))
+  )
+  (wire (pts (xy 83.82 98.425) (xy 83.82 101.6))
+    (stroke (width 0) (type default) (color 0 0 0 0))
+  )
+  (wire (pts (xy 83.82 101.6) (xy 83.82 104.14))
+    (stroke (width 0) (type default) (color 0 0 0 0))
+  )
   (wire (pts (xy 49.53 73.66) (xy 49.53 74.93))
     (stroke (width 0) (type default) (color 0 0 0 0))
   )
-  (wire (pts (xy 46.99 68.58) (xy 109.855 68.58))
+  (wire (pts (xy 116.205 68.58) (xy 160.02 68.58))
+    (stroke (width 0) (type default) (color 0 0 0 0))
+  )
+  (wire (pts (xy 46.99 68.58) (xy 99.695 68.58))
+    (stroke (width 0) (type default) (color 0 0 0 0))
+  )
+  (wire (pts (xy 116.205 81.28) (xy 154.94 81.28))
     (stroke (width 0) (type default) (color 0 0 0 0))
   )
@@
     (pin "3")
   )
+  (symbol (lib_id "Device:D_TVS") (at 99.695 94.615 270) (unit 1)
+    (in_bom yes) (on_board yes)
+    (property "Reference" "D9" (id 0) (at 101.7016 93.4466 90)
+      (effects (font (size 1.27 1.27)) (justify left))
+    )
+    (property "Value" "D_TVS_30V" (id 1) (at 101.7016 95.758 90)
+      (effects (font (size 1.27 1.27)) (justify left))
+    )
+    (property "Footprint" "Diode_SMD:D_SOD-123F" (id 2) (at 99.695 94.615 0)
+      (effects (font (size 1.27 1.27)) hide)
+    )
+    (property "Datasheet" "~" (id 3) (at 99.695 94.615 0)
+      (effects (font (size 1.27 1.27)) hide)
+    )
+    (property "LCSC" "C511921" (id 4) (at 99.695 94.615 0)
+      (effects (font (size 1.27 1.27)) hide)
+    )
+    (property "PartNum" "" (id 5) (at 99.695 94.615 90)
+      (effects (font (size 1.27 1.27)) hide)
+    )
+    (property "Part" "SMFJ30CA" (id 6) (at 99.695 94.615 0)
+      (effects (font (size 1.27 1.27)) hide)
+    )
+    (property "Cost" "0.0436" (id 7) (at 99.695 94.615 0)
+      (effects (font (size 1.27 1.27)) hide)
+    )
+    (pin "1")
+    (pin "2")
+  )
+  (symbol (lib_id "power:GND") (at 83.82 104.14 0) (mirror y) (unit 1)
+    (in_bom yes) (on_board yes)
+    (property "Reference" "#PWR013" (id 0) (at 83.82 110.49 0)
+      (effects (font (size 1.27 1.27)) hide)
+    )
+    (property "Value" "GND" (id 1) (at 83.693 108.5342 0))
+    (property "Footprint" "" (id 2) (at 83.82 104.14 0)
+      (effects (font (size 1.27 1.27)) hide)
+    )
+    (property "Datasheet" "" (id 3) (at 83.82 104.14 0)
+      (effects (font (size 1.27 1.27)) hide)
+    )
+    (pin "1")
+  )
   (symbol (lib_id "power:GND") (at 219.71 46.99 0) (unit 1)
     (in_bom yes) (on_board yes)
@@
     (pin "1")
   )
-  (symbol (lib_id "Device:R") (at 109.855 74.93 0) (unit 1)
-    (in_bom yes) (on_board yes)
-    (property "Reference" "R8" (id 0) (at 104.775 74.93 90))
-    (property "Value" "4.7k" (id 1) (at 107.315 74.93 90))
-    (property "Footprint" "Resistor_SMD:R_0805_2012Metric" (id 2) (at 108.077 74.93 90)
-      (effects (font (size 1.27 1.27)) hide)
-    )
-    (property "Datasheet" "~" (id 3) (at 109.855 74.93 0)
-      (effects (font (size 1.27 1.27)) hide)
-    )
-    (property "LCSC" "C23162" (id 4) (at 109.855 74.93 0)
-      (effects (font (size 1.27 1.27)) hide)
-    )
-    (property "Cost" "0.0009" (id 5) (at 109.855 74.93 0)
-      (effects (font (size 1.27 1.27)) hide)
-    )
-    (property "Part" "0603WAF4701T5E" (id 6) (at 109.855 74.93 0)
+  (symbol (lib_id "Device:R") (at 116.205 74.93 0) (unit 1)
+    (in_bom yes) (on_board yes)
+    (property "Reference" "R8" (id 0) (at 111.125 74.93 90))
+    (property "Value" "4.7k" (id 1) (at 113.665 74.93 90))
+    (property "Footprint" "Resistor_SMD:R_0805_2012Metric" (id 2) (at 114.427 74.93 90)
+      (effects (font (size 1.27 1.27)) hide)
+    )
+    (property "Datasheet" "~" (id 3) (at 116.205 74.93 0)
+      (effects (font (size 1.27 1.27)) hide)
+    )
+    (property "LCSC" "C23162" (id 4) (at 116.205 74.93 0)
+      (effects (font (size 1.27 1.27)) hide)
+    )
+    (property "Cost" "0.0009" (id 5) (at 116.205 74.93 0)
+      (effects (font (size 1.27 1.27)) hide)
+    )
+    (property "Part" "0603WAF4701T5E" (id 6) (at 116.205 74.93 0)
       (effects (font (size 1.27 1.27)) hide)
     )
@@
     (pin "1")
   )
+  (symbol (lib_id "Device:D_TVS") (at 83.82 94.615 270) (unit 1)
+    (in_bom yes) (on_board yes)
+    (property "Reference" "D8" (id 0) (at 85.8266 93.4466 90)
+      (effects (font (size 1.27 1.27)) (justify left))
+    )
+    (property "Value" "D_TVS_30V" (id 1) (at 85.8266 95.758 90)
+      (effects (font (size 1.27 1.27)) (justify left))
+    )
+    (property "Footprint" "Diode_SMD:D_SOD-123F" (id 2) (at 83.82 94.615 0)
+      (effects (font (size 1.27 1.27)) hide)
+    )
+    (property "Datasheet" "~" (id 3) (at 83.82 94.615 0)
+      (effects (font (size 1.27 1.27)) hide)
+    )
+    (property "LCSC" "C511921" (id 4) (at 83.82 94.615 0)
+      (effects (font (size 1.27 1.27)) hide)
+    )
+    (property "PartNum" "" (id 5) (at 83.82 94.615 90)
+      (effects (font (size 1.27 1.27)) hide)
+    )
+    (property "Part" "SMFJ30CA" (id 6) (at 83.82 94.615 0)
+      (effects (font (size 1.27 1.27)) hide)
+    )
+    (property "Cost" "0.0436" (id 7) (at 83.82 94.615 0)
+      (effects (font (size 1.27 1.27)) hide)
+    )
+    (pin "1")
+    (pin "2")
+  )
 )
