File: prototypes/tanksensor/tanksensor/analog_in.kicad_sch (KiCad schematic)
At the start: 12 parts, among them J2 Conn_01x04, J5 Conn_01x04

Commit message: Rev of the tanksensor pcb and esphome config
Parts:
- R1: value 1k -> 6.8k
- R2: value 680 -> 10000
Changed lines of the file:
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@@
     (in_bom yes) (on_board yes)
     (property "Reference" "R1" (id 0) (at 55.88 38.5572 90))
-    (property "Value" "1k" (id 1) (at 55.88 40.8686 90))
+    (property "Value" "6.8k" (id 1) (at 55.88 40.8686 90))
     (property "Footprint" "Resistor_SMD:R_0805_2012Metric" (id 2) (at 55.88 42.037 90)
       (effects (font (size 1.27 1.27)) hide)
@@
       (effects (font (size 1.27 1.27)) (justify left))
     )
-    (property "Value" "680" (id 1) (at 82.7786 50.673 0)
-      (effects (font (size 1.27 1.27)) (justify left))
-    )
+    (property "Value" "10000" (id 1) (at 82.7786 50.673 0)
+      (effects (font (size 1.27 1.27)) (justify left))
+    )
