File: prototypes/tanksensor/tanksensor/tanksensor.kicad_pcb (KiCad board)
At the start: 2 copper layers, 70 x 50 mm, 29 parts, among them J1 Conn_01x02, J2 Conn_01x04, J3 Conn_01x04, J4 Conn_01x03, J5 Conn_01x04, U2 ESP32-DevKitC

Commit message: Rev of the tanksensor pcb and esphome config
Parts:
- added D8: D_TVS_30V, Diode_SMD:D_SOD-123F, B.Cu at (95.2, 48.3)
- added D9: D_TVS_30V, Diode_SMD:D_SOD-123F, B.Cu at (92.7, 50.8)
- R1: value 1k -> 6.8k
- R2: value 680 -> 10000
Routing:
- net GND: track 212.9 -> 220.5 mm
Other:
- board text added: "3"
- board text added: "4"
